File: atmega_isp/atmega_isp.kicad_pcb (KiCad board)
At the start: 2 copper layers, 58.4 x 69.8 mm, 27 parts, among them J1 pwr, J2 analog, J3 ISP, J4 jmp, J5 jmp, J6 PD, J7 FTDI, J8 PB, J9 power, SW1 RST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

Commit message: kicad 6 update
Connections:
- net ~RST renamed ~{RST}
Other:
- net class Default removed
